File: usb_interface.kicad_sch (KiCad schematic)
At the start: 8 parts, among them U2 FUSB302BMPX

Commit message: USB-B micro added
Parts:
- added R27, R28: 0R, Resistor_SMD:R_0402_1005Metric, symbol Device:R
Connections:
- net USB_CC1: now also R28.1
- net USB_CC2: now also R27.1
- new net BYPASS_CC1: R28.2
- new net BYPASS_CC2: R27.2
Other:
- note added: "Bypass of FUSB302BMPX's CC lines"
- note added: "Do not solder, if FUSB302B is used."
