File: obvod.kicad_sch (KiCad schematic)
At the start: 1 part

Commit message: RF_Tx matched to 50ohms
Other:
- added sheet RF (rf.kicad_sch)
Changed lines of the file:
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@@
+	)
+	(sheet
+		(at 107.95 168.91)
+		(size 12.7 17.78)
+		(fields_autoplaced yes)
+		(stroke
+			(width 0.1524)
+			(type solid)
+		)
+		(fill
+			(color 0 0 0 0.0000)
+		)
+		(property "Sheetname" "RF"
+			(at 107.95 168.1984 0)
+			(effects
+				(font
+					(size 1.27 1.27)
+				)
+				(justify left bottom)
+			)
+		)
+		(property "Sheetfile" "rf.kicad_sch"
+			(at 107.95 187.2746 0)
+			(effects
+				(font
+					(size 1.27 1.27)
+				)
+				(justify left top)
+			)
+		)
+		(instances
+			(project "obvod"
+				(path "/e8e834c4-1afb-42f7-b718-3cb720dae1d5"
+					(page "11")
+				)
+			)
+		)
 	)
 	(sheet
