File: hardware/Charger-PowerManagement.kicad_sch (KiCad schematic)
At the start: 16 parts, among them IC2 BQ25302RTER, Q3 DMP2305U-7

Commit message: Battery temperature meter added to MCU
Parts:
- removed RT1: 103AT-2, 103AT2, symbol SamacSys_Parts:103AT-2
Connections:
- net NTC_1: now reaches IC2.7 (TS), R7.2, R8.1
- no-connect marks 2 -> 3
Other:
- moved on the sheet: C4
