File: hardware/Power_Management.kicad_sch (KiCad schematic)
At the start: 15 parts, among them IC2 BQ25302RTER, Q3 DMP2305U-7

Commit message: prevention save
Parts:
- renumbered C3 to C2, C5 to C3, C2 to C4, C4 to C5
Changed lines of the file:
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@@
 		(dnp no)
 		(fields_autoplaced yes)
-		(property "Reference" "C2"
+		(property "Reference" "C4"
 			(at 41.91 95.2499 0)
 			(effects
@@
 			(project "obvod"
 				(path "/e8e834c4-1afb-42f7-b718-3cb720dae1d5/eca20acd-1ab9-4713-a6f3-0ad5760dd36d"
-					(reference "C2")
+					(reference "C4")
 					(unit 1)
 				)
@@
 		(dnp no)
 		(fields_autoplaced yes)
-		(property "Reference" "C5"
+		(property "Reference" "C3"
 			(at 106.68 50.8 90)
 			(effects
@@
 			(project "obvod"
 				(path "/e8e834c4-1afb-42f7-b718-3cb720dae1d5/eca20acd-1ab9-4713-a6f3-0ad5760dd36d"
-					(reference "C5")
+					(reference "C3")
 					(unit 1)
 				)
@@
 		(dnp no)
 		(fields_autoplaced yes)
-		(property "Reference" "C4"
+		(property "Reference" "C5"
 			(at 54.61 129.5399 0)
 			(effects
@@
 			(project "obvod"
 				(path "/e8e834c4-1afb-42f7-b718-3cb720dae1d5/eca20acd-1ab9-4713-a6f3-0ad5760dd36d"
-					(reference "C4")
+					(reference "C5")
 					(unit 1)
 				)
@@
 		(dnp no)
 		(fields_autoplaced yes)
-		(property "Reference" "C3"
+		(property "Reference" "C2"
 			(at 80.01 38.0999 0)
 			(effects
@@
 			(project "obvod"
 				(path "/e8e834c4-1afb-42f7-b718-3cb720dae1d5/eca20acd-1ab9-4713-a6f3-0ad5760dd36d"
-					(reference "C3")
-					(unit 1)
-				)
+					(reference "C2")
+					(unit 1)
+				)

Commit message: Revised and completed BOM
Parts:
- removed D1: LED, LED_SMD:LED_0805_2012Metric, symbol Device:LED
- removed D2: TS4148_RBG, DIOC2012X85N, symbol SamacSys_Parts:TS4148_RBG
- added D1: BAV19WS, Diode_SMD:D_SOD-323, symbol SamacSys_Parts:BAV19WS
- added D2: LO_Q976-PS-25, LEDC1608X80N, symbol SamacSys_Parts:LO_Q976-PS-25
- C3: footprint Capacitor_SMD:C_0805_2012Metric -> Capacitor_SMD:C_0402_1005Metric
- R6: value 150 -> 542; footprint Resistor_SMD:R_0805_2012Metric -> Resistor_SMD:R_0603_1608Metric
- R7: renamed from R5; footprint Resistor_SMD:R_0805_2012Metric -> Resistor_SMD:R_0402_1005Metric
- renumbered C6 to C4, C4 to C5, C5 to C6, R9 to R5, R7 to R8, R8 to R9
Connections:
- net VBUS: now also D1.2 (A)
- net at Q3.1 (G), R5.1: now also D1.1 (K)
- net at R6.2: now also D2.1 (K)
- net at C6.1, IC2.2 (REGN), R8.1: now also D2.2 (A)
Other:
- note added: "Maximum rating of STAT's output sink current is 6 mA R = (5-1.75)/(6e-3) = 542 Ω"
- note added: "^"
- moved on the sheet: R7
