File: hardware/mcu.kicad_sch (KiCad schematic)
At the start: 24 parts, among them U1 STM32H7A3VITx, Y2 ASDDV-8.000MHZ-LR-T

Commit message: Battery temperature meter added to MCU
Parts:
- added R33: 10k, Resistor_SMD:R_0402_1005Metric, symbol Device:R
Connections:
- net GND: now also U1.23 (PA1), R33.1
- net NTC_2: now reaches U1.22 (PA0)
- net NTC_2: now also R33.2
- net 3V3 renamed +3V3
Other:
- note added: "NTC voltage divider"

Commit message: Done?
Connections:
- net COMMAND_DONE: now reaches U1.39 (PE9)
- net nIRQ: now reaches U1.40 (PE10)
- net nSEL: now reaches U1.41 (PE11)
- net SCLK: now reaches U1.42 (PE12)
- net SDO: now reaches U1.43 (PE13)
- net SDI: now reaches U1.44 (PE14)
Changed lines of the file:
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@@
+		)
+	)
+	(hierarchical_label "SDI"
+		(shape output)
+		(at 48.26 93.98 180)
+		(effects
+			(font
+				(size 1.27 1.27)
+			)
+			(justify right)
 		)
 	)
@@
 		)
 	)
+	(hierarchical_label "nSEL"
+		(shape output)
+		(at 48.26 86.36 180)
+		(effects
+			(font
+				(size 1.27 1.27)
+			)
+			(justify right)
+		)
+	)
+	(hierarchical_label "nIRQ"
+		(shape input)
+		(at 48.26 83.82 180)
+		(effects
+			(font
+				(size 1.27 1.27)
+			)
+			(justify right)
+		)
+	)
 	(hierarchical_label "SWDIO"
 		(shape bidirectional)
@@
 		)
 	)
+	(hierarchical_label "SDO"
+		(shape input)
+		(at 48.26 91.44 180)
+		(effects
+			(font
+				(size 1.27 1.27)
+			)
+			(justify right)
+		)
+	)
 	(hierarchical_label "D4"
 		(shape input)
@@
 		)
 	)
+	(hierarchical_label "COMMAND_DONE"
+		(shape input)
+		(at 48.26 81.28 180)
+		(effects
+			(font
+				(size 1.27 1.27)
+			)
+			(justify right)
+		)
+	)
 	(hierarchical_label "D3"
 		(shape input)
@@
 		)
 	)
+	(hierarchical_label "SCLK"
+		(shape output)
+		(at 48.26 88.9 180)
+		(effects
+			(font
+				(size 1.27 1.27)
+			)
+			(justify right)
+		)
+	)

Commit message: Revised and completed BOM
Parts:
- C44: renamed from C20; footprint Capacitor_SMD:C_0603_1608Metric -> Capacitor_SMD:C_0805_2012Metric
- C45: renamed from C21; footprint Capacitor_SMD:C_0603_1608Metric -> Capacitor_SMD:C_0805_2012Metric
- C46: renamed from C16; footprint Capacitor_SMD:C_0805_2012Metric -> Capacitor_SMD:C_0603_1608Metric
- C48: renamed from C18; footprint Capacitor_SMD:C_0805_2012Metric -> Capacitor_SMD:C_0603_1608Metric
- R33: renamed from R11; footprint (none) -> Resistor_SMD:R_0603_1608Metric
- R35: renamed from R29; footprint Resistor_SMD:R_0402_1005Metric -> Capacitor_SMD:C_0603_1608Metric
- R36: renamed from R30; footprint Resistor_SMD:R_0402_1005Metric -> Resistor_SMD:R_0603_1608Metric
- renumbered C9 to C37, C10 to C38, C11 to C39, C12 to C40, C13 to C41, C14 to C42, C15 to C43, C17 to C47, C19 to C49, C25 to C50, C30 to C51, R21 to R32, R23 to R34, R31 to R37, R22 to R38, R33 to R39, Y2 to XTAL
Other:
- moved on the sheet: R39
Changed lines of the file:
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@@
 	(wire
 		(pts
-			(xy 232.41 119.38) (xy 232.41 116.84)
+			(xy 232.41 118.11) (xy 232.41 116.84)
 		)
 		(stroke
@@
 	(wire
 		(pts
-			(xy 232.41 127) (xy 232.41 128.27)
+			(xy 232.41 125.73) (xy 232.41 128.27)
 		)
 		(stroke
@@
 		(dnp no)
 		(fields_autoplaced yes)
-		(property "Reference" "C19"
+		(property "Reference" "C49"
 			(at 238.76 54.6099 0)
 			(effects
@@
 			(project "obvod"
 				(path "/e8e834c4-1afb-42f7-b718-3cb720dae1d5/67c85143-d51e-4a89-ab5a-3edcba0d09a9"
-					(reference "C19")
+					(reference "C49")
 					(unit 1)
 				)
@@
 		(dnp no)
 		(fields_autoplaced yes)
-		(property "Reference" "C16"
+		(property "Reference" "C46"
 			(at 173.99 54.6099 0)
 			(effects
@@
 			)
 		)
-		(property "Footprint" "Capacitor_SMD:C_0805_2012Metric"
+		(property "Footprint" "Capacitor_SMD:C_0603_1608Metric"
 			(at 171.1452 59.69 0)
 			(effects
@@
 			(project "obvod"
 				(path "/e8e834c4-1afb-42f7-b718-3cb720dae1d5/67c85143-d51e-4a89-ab5a-3edcba0d09a9"
-					(reference "C16")
+					(reference "C46")
 					(unit 1)
 				)
@@
 	(symbol
 		(lib_id "Device:R")
-		(at 232.41 123.19 180)
+		(at 232.41 121.92 180)
 		(unit 1)
 		(exclude_from_sim no)
@@
 		(dnp no)
 		(fields_autoplaced yes)
-		(property "Reference" "R33"
-			(at 234.95 121.9199 0)
+		(property "Reference" "R39"
+			(at 234.95 120.6499 0)
 			(effects
 				(font
@@
 		)
 		(property "Value" "10k"
-			(at 234.95 124.4599 0)
+			(at 234.95 123.1899 0)
 			(effects
 				(font
@@
 		)
 		(property "Footprint" "Resistor_SMD:R_0402_1005Metric"
-			(at 234.188 123.19 90)
+			(at 234.188 121.92 90)
 			(effects
 				(font
@@
 		)
 		(property "Datasheet" "~"
-			(at 232.41 123.19 0)
+			(at 232.41 121.92 0)
 			(effects
 				(font
@@
 		)
 		(property "Description" "Resistor"
-			(at 232.41 123.19 0)
+			(at 232.41 121.92 0)
 			(effects
 				(font
@@
 			(project "obvod"
 				(path "/e8e834c4-1afb-42f7-b718-3cb720dae1d5/67c85143-d51e-4a89-ab5a-3edcba0d09a9"
-					(reference "R33")
+					(reference "R39")
 					(unit 1)
 				)
@@
 		(dnp no)
 		(fields_autoplaced yes)
-		(property "Reference" "C25"
+		(property "Reference" "C50"
 			(at 274.32 52.0699 0)
 			(effects
@@
 			(project "obvod"
 				(path "/e8e834c4-1afb-42f7-b718-3cb720dae1d5/67c85143-d51e-4a89-ab5a-3edcba0d09a9"
-					(reference "C25")
+					(reference "C50")
 					(unit 1)
 				)
@@
 		(on_board yes)
 		(dnp no)
-		(property "Reference" "R21"
+		(property "Reference" "R32"
 			(at 161.29 54.61 90)
 			(effects
@@
 			(project "obvod"
 				(path "/e8e834c4-1afb-42f7-b718-3cb720dae1d5/67c85143-d51e-4a89-ab5a-3edcba0d09a9"
-					(reference "R21")
+					(reference "R32")
 					(unit 1)
 				)
@@
 		(dnp no)
 		(fields_autoplaced yes)
-		(property "Reference" "C17"
+		(property "Reference" "C47"
 			(at 187.96 54.6099 0)
 			(effects
@@
 			(project "obvod"
 				(path "/e8e834c4-1afb-42f7-b718-3cb720dae1d5/67c85143-d51e-4a89-ab5a-3edcba0d09a9"
-					(reference "C17")
+					(reference "C47")
 					(unit 1)
 				)
@@
 		(dnp no)
 		(fields_autoplaced yes)
-		(property "Reference" "C9"
+		(property "Reference" "C37"
 			(at 161.29 25.3999 0)
 			(effects
@@
 			(project ""
 				(path "/e8e834c4-1afb-42f7-b718-3cb720dae1d5/67c85143-d51e-4a89-ab5a-3edcba0d09a9"
-					(reference "C9")
+					(reference "C37")
 					(unit 1)
 				)
@@
 		(dnp no)
 		(fields_autoplaced yes)
-		(property "Reference" "C18"
+		(property "Reference" "C48"
 			(at 224.79 54.6099 0)
 			(effects
@@
 			)
 		)
-		(property "Footprint" "Capacitor_SMD:C_0805_2012Metric"
+		(property "Footprint" "Capacitor_SMD:C_0603_1608Metric"
 			(at 221.9452 59.69 0)
 			(effects
@@
 			(project "obvod"
 				(path "/e8e834c4-1afb-42f7-b718-3cb720dae1d5/67c85143-d51e-4a89-ab5a-3edcba0d09a9"
-					(reference "C18")
+					(reference "C48")
 					(unit 1)
 				)
@@
 		(dnp no)
 		(fields_autoplaced yes)
-		(property "Reference" "C30"
+		(property "Reference" "C51"
 			(at 160.02 128.2699 0)
 			(effects
@@
 			(project "obvod"
 				(path "/e8e834c4-1afb-42f7-b718-3cb720dae1d5/67c85143-d51e-4a89-ab5a-3edcba0d09a9"
-					(reference "C30")
+					(reference "C51")
 					(unit 1)
 				)
@@
 		(dnp no)
 		(fields_autoplaced yes)
-		(property "Reference" "C13"
+		(property "Reference" "C41"
 			(at 213.36 25.3999 0)
 			(effects
@@
 			(project "obvod"
 				(path "/e8e834c4-1afb-42f7-b718-3cb720dae1d5/67c85143-d51e-4a89-ab5a-3edcba0d09a9"
-					(reference "C13")
+					(reference "C41")
 					(unit 1)
 				)
@@
 		(on_board yes)
 		(dnp no)
-		(property "Reference" "R11"
+		(property "Reference" "R33"
 			(at 213.36 54.356 90)
 			(effects
@@
 			)
 		)
-		(property "Footprint" ""
+		(property "Footprint" "Resistor_SMD:R_0603_1608Metric"
 			(at 213.36 49.022 90)
 			(effects
@@
 			(project ""
 				(path "/e8e834c4-1afb-42f7-b718-3cb720dae1d5/67c85143-d51e-4a89-ab5a-3edcba0d09a9"
-					(reference "R11")
+					(reference "R33")
 					(unit 1)
 				)
@@
 		(dnp no)
 		(fields_autoplaced yes)
-		(property "Reference" "C15"
+		(property "Reference" "C43"
 			(at 238.76 25.3999 0)
 			(effects
@@
 			(project "obvod"
 				(path "/e8e834c4-1afb-42f7-b718-3cb720dae1d5/67c85143-d51e-4a89-ab5a-3edcba0d09a9"
-					(reference "C15")
+					(reference "C43")
 					(unit 1)
 				)
@@
 		(dnp no)
 		(fields_autoplaced yes)
-		(property "Reference" "R31"
+		(property "Reference" "R37"
 			(at 276.86 82.5499 0)
 			(effects
@@
 			(project "obvod"
 				(path "/e8e834c4-1afb-42f7-b718-3cb720dae1d5/67c85143-d51e-4a89-ab5a-3edcba0d09a9"
-					(reference "R31")
+					(reference "R37")
 					(unit 1)
 				)
@@
 		(dnp no)
 		(fields_autoplaced yes)
-		(property "Reference" "C14"
+		(property "Reference" "C42"
 			(at 226.06 25.3999 0)
 			(effects
@@
 			(project "obvod"
 				(path "/e8e834c4-1afb-42f7-b718-3cb720dae1d5/67c85143-d51e-4a89-ab5a-3edcba0d09a9"
-					(reference "C14")
+					(reference "C42")
 					(unit 1)
 				)
@@
 		(dnp no)
 		(fields_autoplaced yes)
-		(property "Reference" "C12"
+		(property "Reference" "C40"
 			(at 200.66 25.3999 0)
 			(effects
@@
 			(project "obvod"
 				(path "/e8e834c4-1afb-42f7-b718-3cb720dae1d5/67c85143-d51e-4a89-ab5a-3edcba0d09a9"
-					(reference "C12")
+					(reference "C40")
 					(unit 1)
 				)
@@
 		(dnp no)
 		(fields_autoplaced yes)
-		(property "Reference" "C11"
+		(property "Reference" "C39"
 			(at 187.96 25.3999 0)
 			(effects
@@
 			(project "obvod"
 				(path "/e8e834c4-1afb-42f7-b718-3cb720dae1d5/67c85143-d51e-4a89-ab5a-3edcba0d09a9"
-					(reference "C11")
+					(reference "C39")
 					(unit 1)
 				)
@@
 		(dnp no)
 		(fields_autoplaced yes)
-		(property "Reference" "R29"
+		(property "Reference" "R35"
 			(at 205.74 87.6299 0)
 			(effects
@@
 			)
 		)
-		(property "Footprint" "Resistor_SMD:R_0402_1005Metric"
+		(property "Footprint" "Capacitor_SMD:C_0603_1608Metric"
 			(at 201.422 88.9 90)
 			(effects
@@
 			(project "obvod"
 				(path "/e8e834c4-1afb-42f7-b718-3cb720dae1d5/67c85143-d51e-4a89-ab5a-3edcba0d09a9"
-					(reference "R29")
+					(reference "R35")
 					(unit 1)
 				)
@@
 		(dnp no)
 		(fields_autoplaced yes)
-		(property "Reference" "C21"
+		(property "Reference" "C45"
 			(at 274.32 22.8599 0)
 			(effects
@@
 			)
 		)
-		(property "Footprint" "Capacitor_SMD:C_0603_1608Metric"
+		(property "Footprint" "Capacitor_SMD:C_0805_2012Metric"
 			(at 271.4752 27.94 0)
 			(effects
@@
 			(project "obvod"
 				(path "/e8e834c4-1afb-42f7-b718-3cb720dae1d5/67c85143-d51e-4a89-ab5a-3edcba0d09a9"
-					(reference "C21")
+					(reference "C45")
 					(unit 1)
 				)
@@
 		(dnp no)
 		(fields_autoplaced yes)
-		(property "Reference" "C10"
+		(property "Reference" "C38"
 			(at 175.26 25.3999 0)
 			(effects
@@
 			(project "obvod"
 				(path "/e8e834c4-1afb-42f7-b718-3cb720dae1d5/67c85143-d51e-4a89-ab5a-3edcba0d09a9"
-					(reference "C10")
+					(reference "C38")
 					(unit 1)
 				)
@@
 		(dnp no)
 		(fields_autoplaced yes)
-		(property "Reference" "R30"
+		(property "Reference" "R36"
 			(at 218.44 87.6299 0)
 			(effects
@@
 			)
 		)
-		(property "Footprint" "Resistor_SMD:R_0402_1005Metric"
+		(property "Footprint" "Resistor_SMD:R_0603_1608Metric"
 			(at 214.122 88.9 90)
 			(effects
@@
 			(project "obvod"
 				(path "/e8e834c4-1afb-42f7-b718-3cb720dae1d5/67c85143-d51e-4a89-ab5a-3edcba0d09a9"
-					(reference "R30")
+					(reference "R36")
 					(unit 1)
 				)
@@
 		(dnp no)
 		(fields_autoplaced yes)
-		(property "Reference" "R23"
+		(property "Reference" "R34"
 			(at 160.02 91.4399 0)
 			(effects
@@
 			(project "obvod"
 				(path "/e8e834c4-1afb-42f7-b718-3cb720dae1d5/67c85143-d51e-4a89-ab5a-3edcba0d09a9"
-					(reference "R23")
+					(reference "R34")
 					(unit 1)
 				)
@@
 		(dnp no)
 		(fields_autoplaced yes)
-		(property "Reference" "R22"
+		(property "Reference" "R38"
 			(at 276.86 95.2499 0)
 			(effects
@@
 			(project "obvod"
 				(path "/e8e834c4-1afb-42f7-b718-3cb720dae1d5/67c85143-d51e-4a89-ab5a-3edcba0d09a9"
-					(reference "R22")
+					(reference "R38")
 					(unit 1)
 				)
@@
 		(on_board yes)
 		(dnp no)
-		(property "Reference" "Y2"
+		(property "Reference" "XTAL"
 			(at 180.34 112.776 0)
 			(effects
@@
 			(project ""
 				(path "/e8e834c4-1afb-42f7-b718-3cb720dae1d5/67c85143-d51e-4a89-ab5a-3edcba0d09a9"
-					(reference "Y2")
+					(reference "XTAL")
 					(unit 1)
 				)
@@
 		(dnp no)
 		(fields_autoplaced yes)
-		(property "Reference" "C20"
+		(property "Reference" "C44"
 			(at 260.35 22.8599 0)
 			(effects
@@
 			)
 		)
-		(property "Footprint" "Capacitor_SMD:C_0603_1608Metric"
+		(property "Footprint" "Capacitor_SMD:C_0805_2012Metric"
 			(at 257.5052 27.94 0)
 			(effects
@@
 			(project ""
 				(path "/e8e834c4-1afb-42f7-b718-3cb720dae1d5/67c85143-d51e-4a89-ab5a-3edcba0d09a9"
-					(reference "C20")
+					(reference "C44")
 					(unit 1)
 				)
