File: hardware/usb_b.kicad_sch (KiCad schematic)
At the start: 3 parts, among them J4 MCR-B-S-RA-SMT-CS5A-NF-TR, U3 USBLC6-2SC6

Commit message: Revised and completed BOM
Parts:
- renumbered C31 to C15, U3 to IC7, J4 to J3
Other:
- note added: "Configured as device"
- note removed: "Configure as device"
Changed lines of the file:
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@@
 	)
 	(rectangle
-		(start 69.85 72.39)
-		(end 90.17 76.2)
+		(start 68.58 72.39)
+		(end 91.44 76.2)
 		(stroke
 			(width 0)
@@
 		)
 	)
-	(text "Configure as device"
+	(text "Configured as device"
 		(exclude_from_sim no)
 		(at 80.01 74.422 0)
@@
 		(on_board yes)
 		(dnp no)
-		(property "Reference" "U3"
+		(property "Reference" "IC7"
 			(at 106.68 52.07 0)
 			(effects
@@
 			(project ""
 				(path "/e8e834c4-1afb-42f7-b718-3cb720dae1d5/f28d5476-62ad-47ee-95fb-15cfd356e27c"
-					(reference "U3")
+					(reference "IC7")
 					(unit 1)
 				)
@@
 		(on_board yes)
 		(dnp no)
-		(property "Reference" "C31"
+		(property "Reference" "C15"
 			(at 92.71 44.4499 0)
 			(effects
@@
 			(project "obvod"
 				(path "/e8e834c4-1afb-42f7-b718-3cb720dae1d5/f28d5476-62ad-47ee-95fb-15cfd356e27c"
-					(reference "C31")
+					(reference "C15")
 					(unit 1)
 				)
@@
 		(dnp no)
 		(fields_autoplaced yes)
-		(property "Reference" "J4"
+		(property "Reference" "J3"
 			(at 60.96 49.53 0)
 			(effects
@@
 			(project ""
 				(path "/e8e834c4-1afb-42f7-b718-3cb720dae1d5/f28d5476-62ad-47ee-95fb-15cfd356e27c"
-					(reference "J4")
+					(reference "J3")
 					(unit 1)
 				)
