File: hardware/usb_interface.kicad_sch (KiCad schematic)
At the start: 10 parts, among them U2 FUSB302BMPX

Commit message: Battery temperature meter added to MCU
Connections:
- net 3V3 renamed +3V3
Changed lines of the file:
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@@
+	)
+	(junction
+		(at 171.45 50.8)
+		(diameter 0)
+		(color 0 0 0 0)
 	)
 	(junction
@@
 		(color 0 0 0 0)
 	)
-	(junction
-		(at 171.45 50.8)
-		(diameter 0)
-		(color 0 0 0 0)
-	)
 	(wire
 		(pts
@@
 	(wire
 		(pts
+			(xy 171.45 45.72) (xy 171.45 50.8)
+		)
+		(stroke
+			(width 0)
+			(type default)
+		)
+	)
+	(wire
+		(pts
 			(xy 139.7 50.8) (xy 139.7 71.12)
 		)
@@
 		(pts
 			(xy 190.5 118.11) (xy 190.5 97.79)
-		)
-		(stroke
-			(width 0)
-			(type default)
-		)
-	)
-	(wire
-		(pts
-			(xy 182.88 50.8) (xy 171.45 50.8)
 		)
 		(stroke
@@
 		)
 	)
-	(hierarchical_label "3V3"
-		(shape input)
-		(at 182.88 50.8 0)
-		(effects
-			(font
-				(size 1.27 1.27)
-			)
-			(justify left)
-		)
-	)
 	(hierarchical_label "BYPASS_CC2"
 		(shape bidirectional)
@@
 					(unit 1)
 				)
+			)
+		)
+	)
+	(symbol
+		(lib_id "power:+3V3")
+		(at 171.45 45.72 0)
+		(unit 1)
+		(exclude_from_sim no)
+		(in_bom yes)
+		(on_board yes)
+		(dnp no)
+		(property "Reference" "#PWR070"
+			(at 171.45 49.53 0)
+			(effects
+				(font
+					(size 1.27 1.27)
+				)
+				(hide yes)
+			)
+		)
+		(property "Value" "+3V3"
+			(at 170.688 41.656 0)
+			(effects
+				(font
+					(size 1.27 1.27)
+				)
+			)
+		)
+		(property "Footprint" ""
+			(at 171.45 45.72 0)
+			(effects
+				(font
+					(size 1.27 1.27)
+				)
+				(hide yes)
+			)
+		)
+		(property "Datasheet" ""
+			(at 171.45 45.72 0)
+			(effects
+				(font
+					(size 1.27 1.27)
+				)
+				(hide yes)
+			)
+		)
+		(property "Description" "Power symbol creates a global label with name \"+3V3\""
+			(at 171.45 45.72 0)
+			(effects
+				(font
+					(size 1.27 1.27)
+				)
+				(hide yes)
+			)
+		)
+		(pin "1"
+		)
+		(instances
+			(project "obvod"
+				(path "/e8e834c4-1afb-42f7-b718-3cb720dae1d5/fdd3d46b-c5ef-429c-ba04-a467d2c6100e"
+					(reference "#PWR070")
+					(unit 1)
+				)

Commit message: 0R added to RF supply
Parts:
- R27, R28: footprint Resistor_SMD:R_0402_1005Metric -> Resistor_SMD:R_0603_1608Metric
Changed lines of the file:
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@@
 			)
 		)
-		(property "Footprint" "Resistor_SMD:R_0402_1005Metric"
+		(property "Footprint" "Resistor_SMD:R_0603_1608Metric"
 			(at 201.422 93.98 90)
 			(effects
@@
 			)
 		)
-		(property "Footprint" "Resistor_SMD:R_0402_1005Metric"
+		(property "Footprint" "Resistor_SMD:R_0603_1608Metric"
 			(at 188.722 93.98 90)
 			(effects

Commit message: Board connector added
Connections:
- net BYPASS_CC1 renamed BYPASS_CC1_PS
- net BYPASS_CC2 renamed BYPASS_CC2_PS
- net INT_N renamed INT_N_PS
- net USB_SCL renamed USB_SCL_PS
- net USB_SDA renamed USB_SDA_PS
Changed lines of the file:
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@@
 	)
 	(rectangle
-		(start 48.26 82.55)
+		(start 41.91 82.55)
 		(end 78.74 85.09)
 		(stroke
@@
 	(text "Open drain output "
 		(exclude_from_sim no)
-		(at 58.674 83.82 0)
+		(at 52.578 84.074 0)
 		(effects
 			(font
@@
 		)
 	)
-	(hierarchical_label "BYPASS_CC1"
+	(hierarchical_label "BYPASS_CC1_PS"
 		(shape bidirectional)
 		(at 220.98 115.57 0)
@@
 		)
 	)
-	(hierarchical_label "INT_N"
+	(hierarchical_label "INT_N_PS"
 		(shape output)
 		(at 77.47 83.82 180)
@@
 		)
 	)
-	(hierarchical_label "USB_SCL"
+	(hierarchical_label "USB_SCL_PS"
 		(shape input)
 		(at 77.47 81.28 180)
@@
 		)
 	)
-	(hierarchical_label "USB_SDA"
+	(hierarchical_label "USB_SDA_PS"
 		(shape bidirectional)
 		(at 77.47 78.74 180)
@@
 		)
 	)
-	(hierarchical_label "BYPASS_CC2"
+	(hierarchical_label "BYPASS_CC2_PS"
 		(shape bidirectional)
 		(at 220.98 118.11 0)

Commit message: Revised and completed BOM
Parts:
- renumbered C28 to C11, C29 to C12, C26 to C13, C27 to C14, U2 to IC5, R24 to R18, R25 to R19, R26 to R20, R27 to R21, R28 to R22
Changed lines of the file:
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@@
 		(dnp no)
 		(fields_autoplaced yes)
-		(property "Reference" "C26"
+		(property "Reference" "C13"
 			(at 162.56 92.7099 0)
 			(effects
@@
 			(project ""
 				(path "/e8e834c4-1afb-42f7-b718-3cb720dae1d5/fdd3d46b-c5ef-429c-ba04-a467d2c6100e"
-					(reference "C26")
+					(reference "C13")
 					(unit 1)
 				)
@@
 		(dnp no)
 		(fields_autoplaced yes)
-		(property "Reference" "R24"
+		(property "Reference" "R18"
 			(at 88.9 64.7699 0)
 			(effects
@@
 			(project ""
 				(path "/e8e834c4-1afb-42f7-b718-3cb720dae1d5/fdd3d46b-c5ef-429c-ba04-a467d2c6100e"
-					(reference "R24")
+					(reference "R18")
 					(unit 1)
 				)
@@
 		(dnp no)
 		(fields_autoplaced yes)
-		(property "Reference" "R28"
+		(property "Reference" "R22"
 			(at 205.74 92.7099 0)
 			(effects
@@
 			(project "obvod"
 				(path "/e8e834c4-1afb-42f7-b718-3cb720dae1d5/fdd3d46b-c5ef-429c-ba04-a467d2c6100e"
-					(reference "R28")
+					(reference "R22")
 					(unit 1)
 				)
@@
 		(dnp no)
 		(fields_autoplaced yes)
-		(property "Reference" "R27"
+		(property "Reference" "R21"
 			(at 193.04 92.7099 0)
 			(effects
@@
 			(project ""
 				(path "/e8e834c4-1afb-42f7-b718-3cb720dae1d5/fdd3d46b-c5ef-429c-ba04-a467d2c6100e"
-					(reference "R27")
+					(reference "R21")
 					(unit 1)
 				)
@@
 		(dnp no)
 		(fields_autoplaced yes)
-		(property "Reference" "U2"
+		(property "Reference" "IC5"
 			(at 139.3541 91.44 0)
 			(effects
@@
 			(project "obvod"
 				(path "/e8e834c4-1afb-42f7-b718-3cb720dae1d5/fdd3d46b-c5ef-429c-ba04-a467d2c6100e"
-					(reference "U2")
+					(reference "IC5")
 					(unit 1)
 				)
@@
 		(dnp no)
 		(fields_autoplaced yes)
-		(property "Reference" "R25"
+		(property "Reference" "R19"
 			(at 101.6 64.7699 0)
 			(effects
@@
 			(project "obvod"
 				(path "/e8e834c4-1afb-42f7-b718-3cb720dae1d5/fdd3d46b-c5ef-429c-ba04-a467d2c6100e"
-					(reference "R25")
+					(reference "R19")
 					(unit 1)
 				)
@@
 		(dnp no)
 		(fields_autoplaced yes)
-		(property "Reference" "C29"
+		(property "Reference" "C12"
 			(at 175.26 58.4199 0)
 			(effects
@@
 			(project ""
 				(path "/e8e834c4-1afb-42f7-b718-3cb720dae1d5/fdd3d46b-c5ef-429c-ba04-a467d2c6100e"
-					(reference "C29")
+					(reference "C12")
 					(unit 1)
 				)
@@
 		(dnp no)
 		(fields_autoplaced yes)
-		(property "Reference" "C28"
+		(property "Reference" "C11"
 			(at 162.56 58.4199 0)
 			(effects
@@
 			(project "obvod"
 				(path "/e8e834c4-1afb-42f7-b718-3cb720dae1d5/fdd3d46b-c5ef-429c-ba04-a467d2c6100e"
-					(reference "C28")
+					(reference "C11")
 					(unit 1)
 				)
@@
 		(dnp no)
 		(fields_autoplaced yes)
-		(property "Reference" "C27"
+		(property "Reference" "C14"
 			(at 175.26 92.7099 0)
 			(effects
@@
 			(project "obvod"
 				(path "/e8e834c4-1afb-42f7-b718-3cb720dae1d5/fdd3d46b-c5ef-429c-ba04-a467d2c6100e"
-					(reference "C27")
+					(reference "C14")
 					(unit 1)
 				)
@@
 		(dnp no)
 		(fields_autoplaced yes)
-		(property "Reference" "R26"
+		(property "Reference" "R20"
 			(at 114.3 64.7699 0)
 			(effects
@@
 			(project "obvod"
 				(path "/e8e834c4-1afb-42f7-b718-3cb720dae1d5/fdd3d46b-c5ef-429c-ba04-a467d2c6100e"
-					(reference "R26")
-					(unit 1)
-				)
+					(reference "R20")
+					(unit 1)
+				)
