File: hardware/schematics/Power_Management.kicad_sch (KiCad schematic)
At the start: 15 parts, among them IC2 BQ25302RTER, Q3 DMP2305U-7

Commit message: EPS board created
Changed lines of the file:
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@@
 		(dnp no)
 		(property "Reference" "Q3"
-			(at 135.89 40.6401 0)
+			(at 134.62 37.846 0)
 			(effects
 				(font
@@
 		)
 		(property "Value" "DMP2305U-7"
-			(at 135.89 38.1001 0)
+			(at 134.62 40.386 0)
 			(effects
 				(font
