File: hardware/schematics/mcu.kicad_sch (KiCad schematic)
At the start: 25 parts, among them IC9 STM32H7A3VIT6

Commit message: EPS board created
Parts:
- renumbered C37 to C38, C38 to C39, C39 to C40, C40 to C41, C41 to C42, C42 to C43, C43 to C44, C44 to C45, C45 to C46, C46 to C47, C48 to C49, C49 to C50, C50 to C51, C51 to C52
Other:
- note removed: "SMAZAT A OŠETŘIT NEPOTŘEBNÉ PINY!"
Changed lines of the file:
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@@
 		)
 	)
-	(text "SMAZAT A OŠETŘIT NEPOTŘEBNÉ PINY!"
-		(exclude_from_sim no)
-		(at 93.98 186.436 0)
-		(effects
-			(font
-				(size 5 5)
-				(thickness 0.254)
-				(bold yes)
-				(color 255 25 38 1)
-			)
-		)
-	)
 	(text "Use jumpers if \nFUSB302B is used."
 		(exclude_from_sim no)
@@
 		(dnp no)
 		(fields_autoplaced yes)
-		(property "Reference" "C49"
+		(property "Reference" "C50"
 			(at 238.76 54.6099 0)
 			(effects
@@
 			(project "obvod"
 				(path "/e8e834c4-1afb-42f7-b718-3cb720dae1d5/67c85143-d51e-4a89-ab5a-3edcba0d09a9"
-					(reference "C49")
+					(reference "C50")
 					(unit 1)
 				)
@@
 		(dnp no)
 		(fields_autoplaced yes)
-		(property "Reference" "C46"
+		(property "Reference" "C47"
 			(at 173.99 54.6099 0)
 			(effects
@@
 			(project "obvod"
 				(path "/e8e834c4-1afb-42f7-b718-3cb720dae1d5/67c85143-d51e-4a89-ab5a-3edcba0d09a9"
-					(reference "C46")
+					(reference "C47")
 					(unit 1)
 				)
@@
 		(dnp no)
 		(fields_autoplaced yes)
-		(property "Reference" "C50"
+		(property "Reference" "C51"
 			(at 274.32 52.0699 0)
 			(effects
@@
 			(project "obvod"
 				(path "/e8e834c4-1afb-42f7-b718-3cb720dae1d5/67c85143-d51e-4a89-ab5a-3edcba0d09a9"
-					(reference "C50")
+					(reference "C51")
 					(unit 1)
 				)
@@
 		(dnp no)
 		(fields_autoplaced yes)
-		(property "Reference" "C37"
+		(property "Reference" "C38"
 			(at 161.29 25.3999 0)
 			(effects
@@
 			(project ""
 				(path "/e8e834c4-1afb-42f7-b718-3cb720dae1d5/67c85143-d51e-4a89-ab5a-3edcba0d09a9"
-					(reference "C37")
+					(reference "C38")
 					(unit 1)
 				)
@@
 		(dnp no)
 		(fields_autoplaced yes)
-		(property "Reference" "C48"
+		(property "Reference" "C49"
 			(at 224.79 54.6099 0)
 			(effects
@@
 			(project "obvod"
 				(path "/e8e834c4-1afb-42f7-b718-3cb720dae1d5/67c85143-d51e-4a89-ab5a-3edcba0d09a9"
-					(reference "C48")
+					(reference "C49")
 					(unit 1)
 				)
@@
 		(dnp no)
 		(fields_autoplaced yes)
-		(property "Reference" "C51"
+		(property "Reference" "C52"
 			(at 160.02 128.2699 0)
 			(effects
@@
 			(project "obvod"
 				(path "/e8e834c4-1afb-42f7-b718-3cb720dae1d5/67c85143-d51e-4a89-ab5a-3edcba0d09a9"
-					(reference "C51")
+					(reference "C52")
 					(unit 1)
 				)
@@
 		(dnp no)
 		(fields_autoplaced yes)
-		(property "Reference" "C41"
+		(property "Reference" "C42"
 			(at 213.36 25.3999 0)
 			(effects
@@
 			(project "obvod"
 				(path "/e8e834c4-1afb-42f7-b718-3cb720dae1d5/67c85143-d51e-4a89-ab5a-3edcba0d09a9"
-					(reference "C41")
+					(reference "C42")
 					(unit 1)
 				)
@@
 		(dnp no)
 		(fields_autoplaced yes)
-		(property "Reference" "C43"
+		(property "Reference" "C44"
 			(at 238.76 25.3999 0)
 			(effects
@@
 			(project "obvod"
 				(path "/e8e834c4-1afb-42f7-b718-3cb720dae1d5/67c85143-d51e-4a89-ab5a-3edcba0d09a9"
-					(reference "C43")
+					(reference "C44")
 					(unit 1)
 				)
@@
 		(dnp no)
 		(fields_autoplaced yes)
-		(property "Reference" "C42"
+		(property "Reference" "C43"
 			(at 226.06 25.3999 0)
 			(effects
@@
 			(project "obvod"
 				(path "/e8e834c4-1afb-42f7-b718-3cb720dae1d5/67c85143-d51e-4a89-ab5a-3edcba0d09a9"
-					(reference "C42")
+					(reference "C43")
 					(unit 1)
 				)
@@
 		(dnp no)
 		(fields_autoplaced yes)
-		(property "Reference" "C40"
+		(property "Reference" "C41"
 			(at 200.66 25.3999 0)
 			(effects
@@
 			(project "obvod"
 				(path "/e8e834c4-1afb-42f7-b718-3cb720dae1d5/67c85143-d51e-4a89-ab5a-3edcba0d09a9"
-					(reference "C40")
+					(reference "C41")
 					(unit 1)
 				)
@@
 		(dnp no)
 		(fields_autoplaced yes)
-		(property "Reference" "C39"
+		(property "Reference" "C40"
 			(at 187.96 25.3999 0)
 			(effects
@@
 			(project "obvod"
 				(path "/e8e834c4-1afb-42f7-b718-3cb720dae1d5/67c85143-d51e-4a89-ab5a-3edcba0d09a9"
-					(reference "C39")
+					(reference "C40")
 					(unit 1)
 				)
@@
 		(dnp no)
 		(fields_autoplaced yes)
-		(property "Reference" "C45"
+		(property "Reference" "C46"
 			(at 274.32 22.8599 0)
 			(effects
@@
 			(project "obvod"
 				(path "/e8e834c4-1afb-42f7-b718-3cb720dae1d5/67c85143-d51e-4a89-ab5a-3edcba0d09a9"
-					(reference "C45")
+					(reference "C46")
 					(unit 1)
 				)
@@
 		(dnp no)
 		(fields_autoplaced yes)
-		(property "Reference" "C38"
+		(property "Reference" "C39"
 			(at 175.26 25.3999 0)
 			(effects
@@
 			(project "obvod"
 				(path "/e8e834c4-1afb-42f7-b718-3cb720dae1d5/67c85143-d51e-4a89-ab5a-3edcba0d09a9"
-					(reference "C38")
+					(reference "C39")
 					(unit 1)
 				)
@@
 		(dnp no)
 		(fields_autoplaced yes)
-		(property "Reference" "C44"
+		(property "Reference" "C45"
 			(at 260.35 22.8599 0)
 			(effects
@@
 			(project ""
 				(path "/e8e834c4-1afb-42f7-b718-3cb720dae1d5/67c85143-d51e-4a89-ab5a-3edcba0d09a9"
-					(reference "C44")
+					(reference "C45")
 					(unit 1)
 				)
