File: hardware/schematics/usb_b.kicad_sch (KiCad schematic)
At the start: 3 parts, among them IC7 USBLC6-2SC6, J3 MCR-B-S-RA-SMT-CS5A-NF-TR

Commit message: EPS board created
Parts:
- renumbered C15 to C16
Changed lines of the file:
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@@
 		(on_board yes)
 		(dnp no)
-		(property "Reference" "C15"
+		(property "Reference" "C16"
 			(at 92.71 44.4499 0)
 			(effects
@@
 			(project "obvod"
 				(path "/e8e834c4-1afb-42f7-b718-3cb720dae1d5/f28d5476-62ad-47ee-95fb-15cfd356e27c"
-					(reference "C15")
+					(reference "C16")
 					(unit 1)
 				)
