File: hardware/schematics/usb_c.kicad_sch (KiCad schematic)
At the start: 16 parts, among them IC4 TCPP01-M12, J1 UJC-H-G-SMT-2-P6-TR, Q4 STL11N3LLH6

Commit message: EPS board created
Parts:
- renumbered C9 to C10, C10 to C11, C8 to C9
Changed lines of the file:
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@@
 		(dnp no)
 		(fields_autoplaced yes)
-		(property "Reference" "C10"
+		(property "Reference" "C11"
 			(at 151.13 118.1099 0)
 			(effects
@@
 			(project "obvod"
 				(path "/e8e834c4-1afb-42f7-b718-3cb720dae1d5/540adf6e-5b6f-4df1-af18-d763618ddc56"
-					(reference "C10")
+					(reference "C11")
 					(unit 1)
 				)
@@
 		(on_board yes)
 		(dnp no)
-		(property "Reference" "C9"
+		(property "Reference" "C10"
 			(at 138.43 93.9799 0)
 			(effects
@@
 			(project ""
 				(path "/e8e834c4-1afb-42f7-b718-3cb720dae1d5/540adf6e-5b6f-4df1-af18-d763618ddc56"
-					(reference "C9")
+					(reference "C10")
 					(unit 1)
 				)
@@
 		(dnp no)
 		(fields_autoplaced yes)
-		(property "Reference" "C8"
+		(property "Reference" "C9"
 			(at 151.13 71.1199 0)
 			(effects
@@
 			(project ""
 				(path "/e8e834c4-1afb-42f7-b718-3cb720dae1d5/540adf6e-5b6f-4df1-af18-d763618ddc56"
-					(reference "C8")
-					(unit 1)
-				)
+					(reference "C9")
+					(unit 1)
+				)
