File: hardware/schematics/rf.kicad_sch (KiCad schematic)
At the start: 46 parts, among them IC8 SI4468-A2A-IMR, J5 RFPC-SMA28-F, Q6 DMN1008UFDF-7

Commit message: EPS board created
Parts:
- renumbered C16 to C17, C17 to C18, C18 to C19, C19 to C20, C20 to C21, C21 to C22, C22 to C23, C23 to C24, C24 to C25, C25 to C26, C26 to C27, C27 to C28, C28 to C29, C29 to C30, C30 to C31, C31 to C32, C32 to C33, C33 to C34, C34 to C35, C35 to C36, C36 to C37
Changed lines of the file:
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@@
 		(on_board yes)
 		(dnp no)
-		(property "Reference" "C29"
+		(property "Reference" "C30"
 			(at 66.04 99.06 90)
 			(effects
@@
 			(project "obvod"
 				(path "/e8e834c4-1afb-42f7-b718-3cb720dae1d5/21633f2b-133b-44f0-ac2e-c32a8c0675be"
-					(reference "C29")
+					(reference "C30")
 					(unit 1)
 				)
@@
 		(dnp no)
 		(fields_autoplaced yes)
-		(property "Reference" "C25"
+		(property "Reference" "C26"
 			(at 264.16 44.4499 0)
 			(effects
@@
 			(project ""
 				(path "/e8e834c4-1afb-42f7-b718-3cb720dae1d5/21633f2b-133b-44f0-ac2e-c32a8c0675be"
-					(reference "C25")
+					(reference "C26")
 					(unit 1)
 				)
@@
 		(dnp no)
 		(fields_autoplaced yes)
-		(property "Reference" "C35"
+		(property "Reference" "C36"
 			(at 60.96 176.5299 0)
 			(effects
@@
 			(project "obvod"
 				(path "/e8e834c4-1afb-42f7-b718-3cb720dae1d5/21633f2b-133b-44f0-ac2e-c32a8c0675be"
-					(reference "C35")
+					(reference "C36")
 					(unit 1)
 				)
@@
 		(dnp no)
 		(fields_autoplaced yes)
-		(property "Reference" "C34"
+		(property "Reference" "C35"
 			(at 35.56 176.5299 0)
 			(effects
@@
 			(project ""
 				(path "/e8e834c4-1afb-42f7-b718-3cb720dae1d5/21633f2b-133b-44f0-ac2e-c32a8c0675be"
-					(reference "C34")
+					(reference "C35")
 					(unit 1)
 				)
@@
 		(on_board yes)
 		(dnp no)
-		(property "Reference" "C28"
+		(property "Reference" "C29"
 			(at 27.94 99.06 90)
 			(effects
@@
 			(project ""
 				(path "/e8e834c4-1afb-42f7-b718-3cb720dae1d5/21633f2b-133b-44f0-ac2e-c32a8c0675be"
-					(reference "C28")
+					(reference "C29")
 					(unit 1)
 				)
@@
 		(dnp no)
 		(fields_autoplaced yes)
-		(property "Reference" "C17"
+		(property "Reference" "C18"
 			(at 68.58 16.51 90)
 			(effects
@@
 			(project "obvod"
 				(path "/e8e834c4-1afb-42f7-b718-3cb720dae1d5/21633f2b-133b-44f0-ac2e-c32a8c0675be"
-					(reference "C17")
+					(reference "C18")
 					(unit 1)
 				)
@@
 		(on_board yes)
 		(dnp no)
-		(property "Reference" "C27"
+		(property "Reference" "C28"
 			(at 52.832 82.804 90)
 			(effects
@@
 			(project "obvod"
 				(path "/e8e834c4-1afb-42f7-b718-3cb720dae1d5/21633f2b-133b-44f0-ac2e-c32a8c0675be"
-					(reference "C27")
+					(reference "C28")
 					(unit 1)
 				)
@@
 		(dnp no)
 		(fields_autoplaced yes)
-		(property "Reference" "C26"
+		(property "Reference" "C27"
 			(at 276.86 44.4499 0)
 			(effects
@@
 			(project ""
 				(path "/e8e834c4-1afb-42f7-b718-3cb720dae1d5/21633f2b-133b-44f0-ac2e-c32a8c0675be"
-					(reference "C26")
+					(reference "C27")
 					(unit 1)
 				)
@@
 		(on_board yes)
 		(dnp no)
-		(property "Reference" "C33"
+		(property "Reference" "C34"
 			(at 93.98 160.528 90)
 			(effects
@@
 			(project ""
 				(path "/e8e834c4-1afb-42f7-b718-3cb720dae1d5/21633f2b-133b-44f0-ac2e-c32a8c0675be"
-					(reference "C33")
+					(reference "C34")
 					(unit 1)
 				)
@@
 		(on_board yes)
 		(dnp no)
-		(property "Reference" "C18"
+		(property "Reference" "C19"
 			(at 115.57 22.352 90)
 			(effects
@@
 			(project "obvod"
 				(path "/e8e834c4-1afb-42f7-b718-3cb720dae1d5/21633f2b-133b-44f0-ac2e-c32a8c0675be"
-					(reference "C18")
+					(reference "C19")
 					(unit 1)
 				)
@@
 		(on_board yes)
 		(dnp no)
-		(property "Reference" "C30"
+		(property "Reference" "C31"
 			(at 118.11 105.41 0)
 			(effects
@@
 			(project "obvod"
 				(path "/e8e834c4-1afb-42f7-b718-3cb720dae1d5/21633f2b-133b-44f0-ac2e-c32a8c0675be"
-					(reference "C30")
+					(reference "C31")
 					(unit 1)
 				)
@@
 		(dnp no)
 		(fields_autoplaced yes)
-		(property "Reference" "C16"
+		(property "Reference" "C17"
 			(at 27.94 38.0999 0)
 			(effects
@@
 			(project "obvod"
 				(path "/e8e834c4-1afb-42f7-b718-3cb720dae1d5/21633f2b-133b-44f0-ac2e-c32a8c0675be"
-					(reference "C16")
+					(reference "C17")
 					(unit 1)
 				)
@@
 		(dnp no)
 		(fields_autoplaced yes)
-		(property "Reference" "C21"
+		(property "Reference" "C22"
 			(at 186.69 35.5599 0)
 			(effects
@@
 			(project "obvod"
 				(path "/e8e834c4-1afb-42f7-b718-3cb720dae1d5/21633f2b-133b-44f0-ac2e-c32a8c0675be"
-					(reference "C21")
+					(reference "C22")
 					(unit 1)
 				)
@@
 		(on_board yes)
 		(dnp no)
-		(property "Reference" "C36"
+		(property "Reference" "C37"
 			(at 93.98 171.958 90)
 			(effects
@@
 			(project "obvod"
 				(path "/e8e834c4-1afb-42f7-b718-3cb720dae1d5/21633f2b-133b-44f0-ac2e-c32a8c0675be"
-					(reference "C36")
+					(reference "C37")
 					(unit 1)
 				)
@@
 		(dnp no)
 		(fields_autoplaced yes)
-		(property "Reference" "C22"
+		(property "Reference" "C23"
 			(at 276.86 24.1299 0)
 			(effects
@@
 			(project "obvod"
 				(path "/e8e834c4-1afb-42f7-b718-3cb720dae1d5/21633f2b-133b-44f0-ac2e-c32a8c0675be"
-					(reference "C22")
+					(reference "C23")
 					(unit 1)
 				)
@@
 		(on_board yes)
 		(dnp no)
-		(property "Reference" "C19"
+		(property "Reference" "C20"
 			(at 105.41 45.72 0)
 			(effects
@@
 			(project "obvod"
 				(path "/e8e834c4-1afb-42f7-b718-3cb720dae1d5/21633f2b-133b-44f0-ac2e-c32a8c0675be"
-					(reference "C19")
+					(reference "C20")
 					(unit 1)
 				)
@@
 		(dnp no)
 		(fields_autoplaced yes)
-		(property "Reference" "C24"
+		(property "Reference" "C25"
 			(at 251.46 44.4499 0)
 			(effects
@@
 			(project "obvod"
 				(path "/e8e834c4-1afb-42f7-b718-3cb720dae1d5/21633f2b-133b-44f0-ac2e-c32a8c0675be"
-					(reference "C24")
+					(reference "C25")
 					(unit 1)
 				)
@@
 		(dnp no)
 		(fields_autoplaced yes)
-		(property "Reference" "C20"
+		(property "Reference" "C21"
 			(at 161.29 35.5599 0)
 			(effects
@@
 			(project "obvod"
 				(path "/e8e834c4-1afb-42f7-b718-3cb720dae1d5/21633f2b-133b-44f0-ac2e-c32a8c0675be"
-					(reference "C20")
+					(reference "C21")
 					(unit 1)
 				)
@@
 		(dnp no)
 		(fields_autoplaced yes)
-		(property "Reference" "C23"
+		(property "Reference" "C24"
 			(at 238.76 44.4499 0)
 			(effects
@@
 			(project "obvod"
 				(path "/e8e834c4-1afb-42f7-b718-3cb720dae1d5/21633f2b-133b-44f0-ac2e-c32a8c0675be"
-					(reference "C23")
+					(reference "C24")
 					(unit 1)
 				)
@@
 		(on_board yes)
 		(dnp no)
-		(property "Reference" "C32"
+		(property "Reference" "C33"
 			(at 23.114 160.274 90)
 			(effects
@@
 			(project "obvod"
 				(path "/e8e834c4-1afb-42f7-b718-3cb720dae1d5/21633f2b-133b-44f0-ac2e-c32a8c0675be"
-					(reference "C32")
+					(reference "C33")
 					(unit 1)
 				)
@@
 		(on_board yes)
 		(dnp no)
-		(property "Reference" "C31"
+		(property "Reference" "C32"
 			(at 51.562 142.494 90)
 			(effects
@@
 			(project "obvod"
 				(path "/e8e834c4-1afb-42f7-b718-3cb720dae1d5/21633f2b-133b-44f0-ac2e-c32a8c0675be"
-					(reference "C31")
+					(reference "C32")
 					(unit 1)
 				)

Commit message: gitignore added
Other:
- note added: "Limit current to 5mA max. Solder only one of them."
- note added: "or connect jumper to MOSFET's bypass."
- note removed: "Limit current to 5mA max."
- note removed: "Or connect jumper to MOSFET's bypass"
Changed lines of the file:
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@@
 		)
 	)
-	(text "Or connect jumper to \nMOSFET's bypass"
+	(text "or connect jumper to \nMOSFET's bypass."
 		(exclude_from_sim no)
 		(at 58.674 152.654 0)
@@
 		)
 	)
-	(text "Limit current to 5mA max."
+	(text "Limit current to 5mA max.\nSolder only one of them."
 		(exclude_from_sim no)
-		(at 147.574 159.004 0)
+		(at 134.112 158.75 0)
 		(effects
 			(font
 				(size 1.27 1.27)
 			)
+			(justify left)
 		)
 	)
