File: hardware/schematics/usb_interface.kicad_sch (KiCad schematic)
At the start: 10 parts, among them IC5 FUSB302BMPX

Commit message: EPS board created
Parts:
- renumbered C11 to C12, C12 to C13, C13 to C14, C14 to C15
Changed lines of the file:
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@@
 		(dnp no)
 		(fields_autoplaced yes)
-		(property "Reference" "C13"
+		(property "Reference" "C14"
 			(at 162.56 92.7099 0)
 			(effects
@@
 			(project ""
 				(path "/e8e834c4-1afb-42f7-b718-3cb720dae1d5/fdd3d46b-c5ef-429c-ba04-a467d2c6100e"
-					(reference "C13")
+					(reference "C14")
 					(unit 1)
 				)
@@
 		(dnp no)
 		(fields_autoplaced yes)
-		(property "Reference" "C12"
+		(property "Reference" "C13"
 			(at 175.26 58.4199 0)
 			(effects
@@
 			(project ""
 				(path "/e8e834c4-1afb-42f7-b718-3cb720dae1d5/fdd3d46b-c5ef-429c-ba04-a467d2c6100e"
-					(reference "C12")
+					(reference "C13")
 					(unit 1)
 				)
@@
 		(dnp no)
 		(fields_autoplaced yes)
-		(property "Reference" "C11"
+		(property "Reference" "C12"
 			(at 162.56 58.4199 0)
 			(effects
@@
 			(project "obvod"
 				(path "/e8e834c4-1afb-42f7-b718-3cb720dae1d5/fdd3d46b-c5ef-429c-ba04-a467d2c6100e"
-					(reference "C11")
+					(reference "C12")
 					(unit 1)
 				)
@@
 		(dnp no)
 		(fields_autoplaced yes)
-		(property "Reference" "C14"
+		(property "Reference" "C15"
 			(at 175.26 92.7099 0)
 			(effects
@@
 			(project "obvod"
 				(path "/e8e834c4-1afb-42f7-b718-3cb720dae1d5/fdd3d46b-c5ef-429c-ba04-a467d2c6100e"
-					(reference "C14")
-					(unit 1)
-				)
+					(reference "C15")
+					(unit 1)
+				)

Commit message: gitignore added
Other:
- note added: "Solder, if FUSB302B is used."
- note removed: "Do not solder, if FUSB302B is used."
Changed lines of the file:
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@@
 		)
 	)
-	(text "Do not solder, if FUSB302B is used."
+	(text "Solder, if FUSB302B is used."
 		(exclude_from_sim no)
-		(at 61.722 66.04 0)
+		(at 58.674 66.548 0)
 		(effects
 			(font
