File: hardware/PCBs/eps/eps.kicad_sch (KiCad schematic)
At the start: 57 parts, among them IC1 BQ29732DSER, IC2 BQ25302RTER, IC3 XCL240B333FR-G, IC4 TCPP01-M12, IC5 FUSB302BMPX, J1 UJC-H-G-SMT-2-P6-TR, Q1 CSD16406Q3, Q2 CSD16406Q3, Q3 DMP2305U-7, Q4 STL11N3LLH6

Commit message: EPS board created
Parts:
- added J7: PH1-08-UA, HDRV8W64P0X254_1X8_2032X250X888P, symbol SamacSys_Parts:PH1-08-UA
- added J8: PRT-09279, RHDR8W87P0X254_1X8_2087X250X865P, symbol SamacSys_Parts:PRT-09279
- R5: renamed from R9; footprint (none) -> Resistor_SMD:R_0402_1005Metric
- S1: footprint footprints:RA12131100 -> SamacSys_Parts:RA12131100
- renumbered C9 to C10, C10 to C11, C11 to C12, C12 to C13, C13 to C14, C14 to C15, C3 to C2, C5 to C3, C6 to C4, C2 to C5, C4 to C6, C8 to C9, D2 to D1, D1 to D2, R5 to R7, R7 to R8, R8 to R9
Connections:
- net CC1 is gone; now on net USB_CC1: IC4.3 (CC1), R15.1
- net CC2 is gone; now on net USB_CC2: IC4.1 (CC2), R16.1
- net VIN is gone; now on an unnamed net: C7.1, IC3.4 (EN), IC3.6 (VIN)
- net VSYS is gone; now on an unnamed net: C2.1, IC2.16 (PMID), Q3.2 (S)
- net +3V3: now also J8.1
- net ADC_VBUS_PS: now also J7.1
- net BYPASS_CC1_PS: now also J7.6
- net BYPASS_CC2_PS: now also J7.7
- net FLT/_PS: now also J7.2
- net GND: now also J8.8
- net INT_N_PS: now also J7.5
- net NTC_2_PS: now also J7.8
- net USB_SCL_PS: now also J7.4
- net USB_SDA_PS: now also J7.3
- net BAT+: no longer names the net of BAT1.1 (+), BAT2.1 (+), C4.1, IC2.10 (BAT), L1.2, Q3.3 (D), R1.1
- net NTC_1: no longer names the net of IC2.7 (TS), NTC1.2, R8.2, R9.1
- no-connect marks 9 -> 17
Other:
- note added: "<"
- moved on the sheet: BAT1, BAT2, C1, C10, C11, C12, C13, C14, C15, C2, C3, C4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

Commit message: Draft of EPS PCB half-way done
Parts:
- BAT1: footprint 1043 -> SamacSys_Parts:1043
Changed lines of the file:
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@@
 			)
 		)
-		(property "Footprint" "1043"
+		(property "Footprint" "SamacSys_Parts:1043"
 			(at 391.16 336.22 0)
 			(effects

Commit message: PCB-EPS 1/2
Parts:
- added FID1, FID2, FID3: Fiducial, Fiducial:Fiducial_1mm_Mask2mm, symbol Mechanical:Fiducial
- added H1, H2, H3, H4: MountingHole_Pad, MountingHole:MountingHole_3.2mm_M3_Pad, symbol Mechanical:MountingHole_Pad
Connections:
- net GND: now also H1.1, H2.1, H3.1, H4.1
Other:
- note added: "Assembly references"
- note added: "Mounting holes"

Commit message: PCB - EPS done. RF started
Parts:
- added TP1, TP3, TP4, TP5: TestPoint, TestPoint:TestPoint_Plated_Hole_D2.0mm, symbol Connector:TestPoint
- added TP2: TestPoint, TestPoint:TestPoint_THTPad_2.0x2.0mm_Drill1.0mm, symbol Connector:TestPoint
- H1, H2, H3, H4: footprint MountingHole:MountingHole_3.2mm_M3_Pad -> MountingHole:MountingHole_3.2mm_M3_Pad_Via
Connections:
- net +3V3: now also TP5.1
- net GND: now also TP1.1
- net VBUS: now also TP3.1
- net at D3.1 (K), D4.2 (A), J1.A9 (VBUS_1)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: now also TP2.1
- net at BAT1.1 (+), BAT2.1 (+), C4.1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: now also TP4.1
Other:
- note added: "Appply current limited 5V testing source here"
- note added: "Check 3.3 V"
- note added: "Check battery voltage"
- note added: "Check for 5 V here"
