File: hardware/PCBs/eps/eps.kicad_pcb (KiCad board)
At the start: 4 copper layers, 96 x 90 mm, 71 parts, among them IC1 BQ29732DSER, IC2 BQ25302RTER, IC3 XCL240B333FR-G, IC4 TCPP01-M12, IC5 FUSB302BMPX, J1 UJC-H-G-SMT-2-P6-TR, J7 PH1-08-UA, J8 PRT-09279, Q1 CSD16406Q3, Q2 CSD16406Q3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

Commit message: Done? Rev.:1.2
Parts:
- moved J8 2.75 mm to (180.5, 108.5)
- moved J7 2.50 mm to (180.5, 70.5)
- moved R22 0.57 mm to (150.2, 106.5)
Routing:
- net /USB_SDA_PS: track 92.7 -> 102.3 mm
- net /USB_SCL_PS: track 92.2 -> 101.8 mm
- net /BYPASS_CC1_PS: track 40.7 -> 39.2 mm
- net /BYPASS_CC2_PS: track 50.3 -> 49.2 mm
- net /INT_N_PS: track 72.7 -> 71.7 mm
- net /ADC_VBUS_PS: track 69.5 -> 68.4 mm
- net /FLT/_PS: track 92.9 -> 91.9 mm
- net /NTC_2_PS: track 36.6 -> 37.5 mm
- net /USB_CC1: track 47.5 -> 48.1 mm
- net GND: vias 177 -> 178

Commit message: gitignore added
Connections:
- Q1 pad 9: (no net) -> Net-(Q1-D_1)
- Q2 pad 9: (no net) -> Net-(Q1-D_1)
Routing:
- net /NTC_2_PS: track 37.5 -> 34.6 mm
- net GND: track 32.5 -> 29.6 mm, vias 178 -> 202
- net /FLT/_PS: track 91.9 -> 90.8 mm
Other:
- board text added: "3V3"
- board text added: "ADC_VBUS"
- board text added: "CC1"
- board text added: "CC2"
- board text added: "FLT/"
- board text added: "INT_N"
- board text added: "NTC"
- board text added: "SCL"
- board text added: "SDA"
- board text removed: "3.3 V"
