File: hardware/PCBs/mcu/mcu.kicad_pcb (KiCad board)
At the start: 4 copper layers, 96 x 90 mm, 43 parts, among them IC6 ESDALC6V1W5, IC7 USBLC6-2SC6, IC9 STM32H7A3VIT6, J1 61301611821, J2 22-16-2060, J3 MCR-B-S-RA-SMT-CS5A-NF-TR, J4 RS2-18-G, Q5 DMN1008UFDF-7

Commit message: Done? Rev.:1.2
Parts:
- moved R35 14.3 mm to (143.0, 66.7)
- moved R36 12.1 mm to (138.5, 65.0), turned to -90 degrees
Connections:
- IC9 pad 3: /D4 -> unconnected-(IC9-PE4-Pad3)
- IC9 pad 4: /D6 -> unconnected-(IC9-PE5-Pad4)
- IC9 pad 5: /D7 -> unconnected-(IC9-PE6-Pad5)
- IC9 pad 52: /D2 -> unconnected-(IC9-PB13-Pad52)
- IC9 pad 69: /D1 -> unconnected-(IC9-PA10-Pad69)
- IC9 pad 92: /D5 -> unconnected-(IC9-PB6-Pad92)
- IC9 pad 97: /D2 -> unconnected-(IC9-PE0-Pad97)
- IC9 pad 98: /D3 -> unconnected-(IC9-PE1-Pad98)
Routing:
- net /SDI: track 8.33 -> 91.2 mm
- net /SCLK: track 8.33 -> 90.8 mm
- net /FLT/: track 8.33 -> 90.0 mm, vias 0 -> 2
- net /SDO: track 8.33 -> 89.0 mm, vias 0 -> 2
- net /ADC_VBUS: track 3.33 -> 81.2 mm, vias 0 -> 2
- net /nSEL: track 8.33 -> 79.9 mm
- net /CC2: track 3.33 -> 74.2 mm
- net /CC1: track 3.33 -> 72.6 mm
- net /INT_N: track 3.33 -> 71.7 mm
- net /D0: track 3.09 -> 68.3 mm
- net /D1: track 4.34 -> 64.3 mm, vias 2 -> 4
- net /D2: track 9.42 -> 67.0 mm
- net /CAM_SDA: track 44.6 -> 102.0 mm, vias 2 -> 4
- net /nIRQ: track 8.33 -> 64.9 mm, vias 0 -> 2
- net /D3: track 10.7 -> 65.4 mm, vias 2 -> 4
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- added copper zone on B.Cu, net GND

Commit message: gitignore added
Parts:
- R33: value 47R -> 0R
- moved FID2 126.1 mm to (165.5, 62.0)
- moved FID3 84.4 mm to (80.5, 125.0)
- moved FID1 44.2 mm to (80.5, 62.0)
- renumbered R2 to R34
Routing:
- net /PCLK: track 67.6 -> 68.6 mm
- net GND: vias 144 -> 151
Other:
- board text added: "ADC_VBUS"
- board text added: "CAM_SCL"
- board text added: "CAM_SDA"
- board text added: "CC1"
- board text added: "CC2"
- board text added: "DONE"
- board text added: "FLT/"
- board text added: "INT_N"
- board text added: "J1"
- board text added: "J2"
- board text added: "Jan Kusak"
- board text added: "NTC_2"
- board text added: "Q5"
- board text added: "SCLK"
- board text added: "SDI"
- board text added: "SDO"
- board text added: "nIRQ"
- board text added: "nSEL"
