File: hardware/PCBs/mcu/mcu.kicad_sch (KiCad schematic)
At the start: 43 parts, among them IC6 ESDALC6V1W5, IC7 USBLC6-2SC6, IC9 STM32H7A3VIT6, J1 61301611821, J2 22-16-2060, J3 MCR-B-S-RA-SMT-CS5A-NF-TR, J4 RS2-18-G, Q5 DMN1008UFDF-7

Commit message: Done? Rev.:1.2
Connections:
- net D1: no longer IC9.69 (PA10)
- net D2: no longer IC9.52 (PB13), IC9.97 (PE0)
- net D3: no longer IC9.98 (PE1)
- net D4: no longer IC9.3 (PE4)
- net D5: no longer IC9.92 (PB6)
- net D6: no longer IC9.4 (PE5)
- net D7: no longer IC9.5 (PE6)
- no-connect marks 39 -> 47
Changed lines of the file:
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@@
 	)
 	(no_connect
+		(at 179.07 76.2)
+	)
+	(no_connect
 		(at 179.07 60.96)
 	)
@@
 	)
 	(no_connect
+		(at 224.79 68.58)
+	)
+	(no_connect
 		(at 179.07 147.32)
 	)
@@
 	)
 	(no_connect
+		(at 179.07 78.74)
+	)
+	(no_connect
 		(at 224.79 96.52)
 	)
@@
 	)
 	(no_connect
+		(at 224.79 101.6)
+	)
+	(no_connect
 		(at 224.79 91.44)
 	)
@@
 	)
 	(no_connect
+		(at 179.07 68.58)
+	)
+	(no_connect
+		(at 179.07 66.04)
+	)
+	(no_connect
 		(at 179.07 114.3)
 	)
@@
 	)
 	(no_connect
+		(at 224.79 119.38)
+	)
+	(no_connect
 		(at 224.79 50.8)
 	)
@@
 	)
 	(no_connect
+		(at 179.07 81.28)
+	)
+	(no_connect
 		(at 179.07 111.76)
 	)
@@
 		)
 	)
-	(hierarchical_label "D2"
-		(shape input)
-		(at 179.07 66.04 180)
-		(effects
-			(font
-				(size 1.27 1.27)
-			)
-			(justify right)
-		)
-	)
 	(hierarchical_label "NTC_2"
 		(shape input)
@@
 		)
 	)
-	(hierarchical_label "D5"
-		(shape input)
-		(at 224.79 101.6 0)
-		(effects
-			(font
-				(size 1.27 1.27)
-			)
-			(justify left)
-		)
-	)
-	(hierarchical_label "D1"
-		(shape input)
-		(at 224.79 68.58 0)
-		(effects
-			(font
-				(size 1.27 1.27)
-			)
-			(justify left)
-		)
-	)
-	(hierarchical_label "D2"
-		(shape input)
-		(at 224.79 119.38 0)
-		(effects
-			(font
-				(size 1.27 1.27)
-			)
-			(justify left)
-		)
-	)
 	(hierarchical_label "nSEL"
 		(shape output)
@@
 	)
 	(hierarchical_label "D6"
-		(shape input)
-		(at 179.07 78.74 180)
-		(effects
-			(font
-				(size 1.27 1.27)
-			)
-			(justify right)
-		)
-	)
-	(hierarchical_label "D6"
 		(shape output)
 		(at 142.24 232.41 180)
@@
 		)
 	)
-	(hierarchical_label "D3"
-		(shape input)
-		(at 179.07 68.58 180)
-		(effects
-			(font
-				(size 1.27 1.27)
-			)
-			(justify right)
-		)
-	)
 	(hierarchical_label "D5"
 		(shape output)
@@
 		)
 	)
-	(hierarchical_label "D7"
-		(shape input)
-		(at 179.07 81.28 180)
-		(effects
-			(font
-				(size 1.27 1.27)
-			)
-			(justify right)
-		)
-	)
 	(hierarchical_label "nSEL"
 		(shape input)
@@
 		(effects
 			(font
-				(size 1.27 1.27)
-			)
-			(justify right)
-		)
-	)
-	(hierarchical_label "D4"
-		(shape input)
-		(at 179.07 76.2 180)
-		(effects
-			(font

Commit message: gitignore added
Parts:
- C16, C39, C40, C41, C42, C43, C44, C47, C50, C51: LCSC part number (none) -> C131394; Manufacturer_Name (none) -> YAGEO; Manufacturer_Part_Number (none) -> CC0402KRX7R9BB104; Mouser Link (none) -> https://cz.mouser.com/ProductDetail/YAGEO/CC0402KRX7R9BB104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; Mouser Part Number (none) -> 603-CC402KRX7R9BB104
- C38: LCSC part number (none) -> C2203601; Manufacturer_Name (none) -> Murata Electronics; Manufacturer_Part_Number (none) -> GRM21BR71C475KE51K; Mouser Link (none) -> https://cz.mouser.com/ProductDetail/Murata-Electronics/GRM2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; Mouser Part Number (none) -> 81-GRM21BR71C475KE1K
- C45, C46: LCSC part number (none) -> C19110; Manufacturer_Name (none) -> Samsung Electro-Mechanics; Manufacturer_Part_Number (none) -> CL21B225KAFNNNE; Mouser Link (none) -> https://cz.mouser.com/ProductDetail/Samsung-Electro-Mechani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; Mouser Part Number (none) -> 187-CL21B225KAFNNNE
- C47, C49: LCSC part number (none) -> C5768807; Manufacturer_Name (none) -> TAIYO YUDEN; Manufacturer_Part_Number (none) -> MLAST168SB7105KTNA01; Mouser Link (none) -> https://cz.mouser.com/ProductDetail/TAIYO-YUDEN/MLAST168SB7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; Mouser Part Number (none) -> 963-MLAST168SB7105KT
- C52: LCSC part number (none) -> C272878; Manufacturer_Name (none) -> YAGEO; Manufacturer_Part_Number (none) -> CC0402JRX7R9BB103; Mouser Link (none) -> https://cz.mouser.com/ProductDetail/YAGEO/CC0402JRX7R9BB103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; Mouser Part Number (none) -> 603-CC402JRX7R9BB103
- D5: LCSC part number (none) -> C283619; Mouser Link (none) -> https://cz.mouser.com/ProductDetail/STMicroelectronics/SMLV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
- IC6: LCSC part number (none) -> C703691; Mouser Link (none) -> https://cz.mouser.com/ProductDetail/STMicroelectronics/ESDA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
- IC7: LCSC part number (none) -> C7519; Manufacturer_Name (none) -> STMicroelectronics; Manufacturer_Part_Number (none) -> USBLC6-2SC6; Mouser Link (none) -> https://cz.mouser.com/ProductDetail/STMicroelectronics/USBL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; Mouser Part Number (none) -> 511-USBLC6-2SC6
- IC9: LCSC part number (none) -> C730222; Manufacturer_Name (none) -> STMicroelectronics; Manufacturer_Part_Number (none) -> STM32H7A3VIT6; Mouser Link (none) -> https://cz.mouser.com/ProductDetail/STMicroelectronics/STM3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; Mouser Part Number (none) -> 511-STM32H7A3VIT6
- J1: Mouser Link (none) -> https://cz.mouser.com/ProductDetail/Same-Sky/UJC-H-G-SMT-2-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; now left out of the parts list
- J2: Mouser Link (none) -> https://cz.mouser.com/ProductDetail/Molex/22-16-2060?qs=rYI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; now left out of the parts list
- J3: Manufacturer_Name (none) -> Adam Tech; Manufacturer_Part_Number (none) -> MCR-B-S-RA-SMT-CS5A-NF-T/R; Mouser Link (none) -> https://cz.mouser.com/ProductDetail/Adam-Tech/MCR-B-S-RA-SM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; Mouser Part Number (none) -> 737-RBSRASMTCS5ANFTR; now left out of the parts list
- J4: Mouser Link (none) -> https://cz.mouser.com/ProductDetail/Adam-Tech/RS2-18-G?qs=H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; Mouser Part Number (none) -> 737-RS2-18-G; now left out of the parts list
- Q5: Mouser Link (none) -> https://cz.mouser.com/ProductDetail/Diodes-Incorporated/DMN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; now left out of the parts list
- R21: LCSC part number (none) -> C705666; Manufacturer_Name (none) -> Susumu; Manufacturer_Part_Number (none) -> RT0402DRD07100KL; Mouser Link (none) -> https://cz.mouser.com/ProductDetail/Susumu/RR0510P-104-D?qs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; Mouser Part Number (none) -> 754-RR0510P-104D
- R22: LCSC part number (none) -> C2902856; Manufacturer_Name (none) -> Panasonic; Manufacturer_Part_Number (none) -> ERA-3AEB1690V; Mouser Link (none) -> https://cz.mouser.com/ProductDetail/Panasonic/ERA-3AEB1690V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; Mouser Part Number (none) -> 667-ERA-3AEB1690V
- R32, R36: LCSC part number (none) -> C100044; Manufacturer_Name (none) -> Vishay / Dale; Manufacturer_Part_Number (none) -> CRCW06030000Z0EE; Mouser Link (none) -> https://cz.mouser.com/ProductDetail/Vishay-Dale/CRCW0603000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; Mouser Part Number (none) -> 71-CRCW06030000Z0EE
- R33: value 47R -> 0R; LCSC part number (none) -> C100044; Manufacturer_Name (none) -> Susumu; Manufacturer_Part_Number (none) -> RG1608P-470-D-T5; Mouser Link (none) -> https://cz.mouser.com/ProductDetail/Susumu/RG1608P-470-D-T5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; Mouser Part Number (none) -> 754-RG1608P-470DT5
- R34: renamed from R2; LCSC part number (none) -> C190095; Manufacturer_Name (none) -> YAGEO; Manufacturer_Part_Number (none) -> RT0402BRD0710KL; Mouser Link (none) -> https://cz.mouser.com/ProductDetail/YAGEO/RT0402BRD0710KL?q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; Mouser Part Number (none) -> 603-RT0402BRD0710KL
- R35: footprint Capacitor_SMD:C_0603_1608Metric -> Resistor_SMD:R_0603_1608Metric; LCSC part number (none) -> C100044; Manufacturer_Name (none) -> Vishay / Dale; Manufacturer_Part_Number (none) -> CRCW06030000Z0EE; Mouser Link (none) -> https://cz.mouser.com/ProductDetail/Vishay-Dale/CRCW0603000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; Mouser Part Number (none) -> 71-CRCW06030000Z0EE
- R37: Manufacturer_Name (none) -> Susumu; Manufacturer_Part_Number (none) -> RR0510P-1691-D; Mouser Link (none) -> https://cz.mouser.com/ProductDetail/Susumu/RR0510P-1691-D?q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; Mouser Part Number (none) -> 754-RR0510P-1691D; now left out of the parts list
- R38: LCSC part number (none) -> C2689454; Manufacturer_Name (none) -> Susumu; Manufacturer_Part_Number (none) -> RR0510P-332-D; Mouser Link (none) -> https://cz.mouser.com/ProductDetail/Susumu/RR0510P-332-D?qs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; Mouser Part Number (none) -> 754-RR0510P-332D
- R39: LCSC part number (none) -> C190095; Manufacturer_Name (none) -> YAGEO; Manufacturer_Part_Number (none) -> RT0402BRD0710KL; Mouser Link (none) -> https://cz.mouser.com/ProductDetail/YAGEO/RT0402BRD0710KL?q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; Mouser Part Number (none) -> 603-RT0402BRD0710KL
- XTAL: Mouser Link (none) -> https://cz.mouser.com/ProductDetail/ABRACON/ASDDV-8.000MHZ-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; now left out of the parts list
