File: hardware/PCBs/rf/rf.kicad_sch (KiCad schematic)
At the start: 54 parts, among them IC8 SI4468-A2A-IMR, J1 PH1-08-UA, J5 RFPC-SMA28-F, Q6 DMN1008UFDF-7

Commit message: Matlab added
Parts:
- R24: value 178 -> 110
- renumbered TCXO to TCXO1
Changed lines of the file:
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@@
 		(dnp no)
 		(fields_autoplaced yes)
-		(property "Reference" "TCXO"
+		(property "Reference" "TCXO1"
 			(at 44.45 16.51 0)
 			(effects
@@
 			)
 		)
-		(property "Value" "178"
+		(property "Value" "110"
 			(at 24.13 73.6599 0)
 			(effects
